File: FirstBoard/FirstBoard.kicad_pcb (KiCad board)
At the start: 2 copper layers, 21 parts, among them J0 Battery, J1 MPU0, J10 MPU9, J11 MPU10, J12 MPU11, J140,208 MPU12, J15 SD_CARD, J2 MPU1, J3 MPU3, J4 MPU3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

Commit message: changing number of pins on MPU connector
Parts:
- J1, J10, J11, J12, J2, J3, J4, J5, J6, J7, J8, J9: footprint Connector_PinHeader_2.54mm:PinHeader_1x06_P2.54mm_Vertical -> Connector_PinHeader_2.54mm:PinHeader_1x08_P2.54mm_Vertical
- J13: renamed from J140,208; footprint Connector_PinHeader_2.54mm:PinHeader_1x06_P2.54mm_Vertical -> Connector_PinHeader_2.54mm:PinHeader_1x08_P2.54mm_Vertical
- moved J13 5.27 mm to (20.5, 38.6)
- moved J1 5.24 mm to (145.5, 145.4)
- moved J2 5.24 mm to (145.5, 131.3)
- moved J3 5.24 mm to (145.5, 117.4)
- moved J4 5.24 mm to (145.5, 103.6)
- moved J5 5.24 mm to (145.5, 89.8)
- moved J6 5.24 mm to (145.5, 73.9)
- moved J7 5.24 mm to (145.5, 58.3)
- moved J10 5.22 mm to (62.7, 38.6)
- moved J11 5.22 mm to (49.5, 38.6)
- moved J12 5.22 mm to (35.9, 38.6)
- moved J8 5.22 mm to (94.4, 38.6)
- moved J9 5.22 mm to (81.5, 38.6)
- moved J15 2.15 mm to (130.0, 197.5)
Connections:
- J1 pad 5: AD0_0 -> unconnected-(J1-Pad5)
- J1 pad 6: INT -> unconnected-(J1-Pad6)
- J10 pad 5: AD0_9 -> unconnected-(J10-Pad5)
- J11 pad 5: AD0_10 -> unconnected-(J11-Pad5)
- J12 pad 5: AD0_11 -> unconnected-(J12-Pad5)
- J13 pad 5: AD0_12 -> unconnected-(J13-Pad5)
- J15 pad 1: GND -> 3v3
- J15 pad 2: 3v3 -> SS
- J15 pad 3: MISO -> MOSI
- J15 pad 4: MOSI -> SCK
- J15 pad 5: SCK -> MISO
- J15 pad 6: SS -> GND
- J2 pad 5: AD0_1 -> unconnected-(J2-Pad5)
- J3 pad 5: AD0_2 -> unconnected-(J3-Pad5)
- J4 pad 5: AD0_3 -> unconnected-(J4-Pad5)
- J5 pad 5: AD0_4 -> unconnected-(J5-Pad5)
- J6 pad 5: AD0_5 -> unconnected-(J6-Pad5)
- J7 pad 5: AD0_6 -> unconnected-(J7-Pad5)
- J8 pad 5: AD0_7 -> unconnected-(J8-Pad5)
- J9 pad 5: AD0_8 -> unconnected-(J9-Pad5)
Routing:
- net 3v3: track 516.6 -> 628.4 mm
- net SCL: track 256.5 -> 283.8 mm
- net SDA: track 244.2 -> 255.3 mm
- net SS: track 165.9 -> 174.9 mm
- net SCK: track 164.2 -> 165.5 mm
- net MOSI: track 154.3 -> 155.2 mm
- net AD0_4: track 39.0 -> 39.9 mm
- net GND: vias 1 -> 2

Commit message: ending the first PCB done-v1
Routing:
- net MISO: track 157.3 -> 155.3 mm
- net 3v3: track 628.4 -> 629.1 mm
